Commit message: Changes to add the Kinect RGB-D

File: map_my_q802/urdf/q802_skid_steer_bot.xacro (robot description, xacro)
@@ -198,6 +198,14 @@
   </joint>
   <!-- SENSORS -->
-  <!-- Camera sensor -->
-  <link name="camera">
+  <!-- RGB-D (Kinect) Camera sensor linked to camera_link -->
+  <joint name="camera_optical_joint" type="fixed">
+    <origin xyz="0 0 0" rpy="-1.5707 0 -1.5707"/>
+    <parent link="camera_link"/>
+    <child link="camera_link_optical"/>
+  </joint>
+  <link name="camera_link_optical">
+  </link>
+  <!-- Orig Camera sensor -->
+  <link name="camera_link">
   <box_inertia m="0.1" x="0.05" y="0.05" d="0.05"/>
     <inertial>
@@ -225,5 +233,5 @@
   <joint type="fixed" name="camera_joint">
     <origin xyz="0.3 0 0" rpy="0 0 0"/>
-    <child link="camera"/>
+    <child link="camera_link"/>
     <parent link="chassis"/>
     <axis xyz="0 1 0" rpy="0 0 0"/>
